File: NRF24.kicad_pcb (KiCad board)
At the start: 4 copper layers, 35.9 x 36.4 mm, 40 parts, among them J1 Conn_ARM_JTAG_SWD_10, J2 SMA, Q1 PMF170XP, Q2 PMF170XP, U1 Si7021-A20, U2 STM32L031G6Ux, U3 nRF24L01P, Y1 16MHz

Commit message: Minor changes
Parts:
- moved J1 11.5 mm to (156.0, 86.2)
- moved C10 0.25 mm to (181.2, 84.0)
- moved C11 0.25 mm to (183.2, 84.0)
- moved C9 0.25 mm to (183.2, 83.0)
Routing:
- net VCC: track 0.00 -> 7.58 mm, vias 0 -> 2
- net GND: track 0.00 -> 7.06 mm, vias 0 -> 5
- net Net-(C16-Pad1): track 0.00 -> 6.48 mm
- net Net-(C13-Pad1): track 0.00 -> 4.64 mm
- net Net-(L2-Pad2): track 0.00 -> 2.43 mm
- net Net-(L2-Pad1): track 0.00 -> 2.42 mm
- net Net-(C11-Pad2): track 0.00 -> 2.42 mm
- net Net-(C10-Pad2): track 0.00 -> 1.42 mm
- net Net-(C16-Pad2): track 0.00 -> 1.03 mm
Other:
- net class Default: clearance 0.2 -> 0.1; trace_width 0.25 -> 0.1
- rule trace_clearance: 0.2 -> 0.1
- rule trace_min: 0.2 -> 0.1

Commit message: Layout
Parts:
- added C18: 10nF, Capacitor_SMD:C_0402_1005Metric, F.Cu at (181.8, 90.5)
- J1: moved to F.Cu
- J2: footprint ak:SMA_Samtec_SMA-J-P-H-ST-EM1_EdgeMount -> Connector_Coaxial:SMA_Samtec_SMA-J-P-H-ST-EM1_EdgeMount
- moved LD1 24.7 mm to (192.5, 78.5)
- moved R7 24.7 mm to (192.5, 75.2)
- moved R8 24.7 mm to (187.5, 74.5)
- moved R9 24.7 mm to (188.5, 74.5)
- moved C3 24.6 mm to (176.2, 76.0), turned to 0 degrees
- moved J1 23.0 mm to (175.5, 98.5), turned to 90 degrees
- moved U1 20.9 mm to (175.8, 78.8), turned to 90 degrees
- moved C2 13.7 mm to (176.0, 93.8), turned to 180 degrees
- moved C7 12.4 mm to (177.2, 91.8), turned to 0 degrees
- moved C1 12.0 mm to (173.2, 91.8), turned to 180 degrees
- moved C6 10.5 mm to (176.8, 90.5), turned to 0 degrees
- moved C4 9.96 mm to (173.5, 90.5), turned to 180 degrees
- moved R3 7.20 mm to (172.0, 87.8)
- moved U2 5.59 mm to (175.5, 87.2), turned to 90 degrees
- moved C8 3.69 mm to (184.2, 73.5)
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Connections:
- net Net-(C11-Pad2) renamed +VSW
- U2 pad 10: /SPI_CSN -> Net-(U2-Pad10)
- U2 pad 14: /NRF_PWR -> /NRF_CSN
- U2 pad 15: Net-(U2-Pad15) -> /NRF_CE
- U2 pad 18: Net-(U2-Pad18) -> /NRF_PWR
- U2 pad 8: /NRF_CE -> /NRF_IRQ
- U2 pad 9: /NRF_IRQ -> Net-(U2-Pad9)
- U3 pad 2: /SPI_CSN -> /NRF_CSN
Routing:
- net /SWDIO: track 0.00 -> 17.2 mm
- net /SWCLK: track 0.00 -> 16.6 mm
- net /NRST: track 0.00 -> 9.30 mm
- net Net-(C12-Pad1): track 0.00 -> 6.90 mm
- net GND: track 7.06 -> 13.7 mm, vias 5 -> 11
- net Net-(C14-Pad1): track 0.00 -> 5.25 mm
- net /SPI_MISO: track 0.00 -> 4.99 mm
- net /SPI_SCK: track 0.00 -> 4.79 mm, vias 0 -> 2
- net /NRF_IRQ: track 0.00 -> 4.18 mm
- net /NRF_CE: track 0.00 -> 3.98 mm
- net /SPI_MOSI: track 0.00 -> 3.75 mm
- net /NRF_CSN: track 0.00 -> 3.53 mm
- net +VSW: track 2.42 -> 4.69 mm, vias 0 -> 1
- net Net-(R6-Pad1): track 0.00 -> 2.21 mm
- net /BOOT0: track 0.00 -> 1.57 mm
- added copper zone on In2.Cu, net +VSW
- added copper zone on In1.Cu, net GND
- added copper zone on In2.Cu, net VCC
Other:
- net class Default: clearance 0.1 -> 0.15; trace_width 0.1 -> 0.15
- rule trace_clearance: 0.1 -> 0.15
- rule via_min_drill: 0.3 -> 0.25
- rule via_min_size: 0.4 -> 0.5

Commit message: Layout
Parts:
- added C19: TBD, Capacitor_SMD:C_0603_1608Metric, F.Cu at (184.8, 79.9)
- LD1: value GREEN -> BLUE; footprint LED_SMD:LED_0603_1608Metric -> LED_SMD:LED_0402_1005Metric
- Q1, Q2: value PMF170XP -> NTK3139P; footprint Package_TO_SOT_SMD:SOT-323_SC-70 -> Package_TO_SOT_SMD:SOT-723
- R7: value 2k2 -> 10R; footprint Resistor_SMD:R_0603_1608Metric -> Resistor_SMD:R_0402_1005Metric
- moved R8 24.7 mm to (173.3, 94.7)
- moved R9 24.7 mm to (174.3, 94.7)
- moved R7 22.3 mm to (179.1, 93.1), turned to 270 degrees
- moved LD1 18.3 mm to (179.1, 90.9), turned to 90 degrees
- moved C8 6.49 mm to (183.2, 79.9)
- moved R5 6.21 mm to (181.9, 79.4)
- moved J1 5.84 mm to (181.2, 99.5), turned to 180 degrees
- moved R4 5.69 mm to (178.9, 79.4)
- moved Q1 5.65 mm to (180.4, 79.4)
- moved C3 4.99 mm to (172.9, 79.7), turned to 90 degrees
- moved R2 4.37 mm to (178.5, 82.0), turned to 90 degrees
- moved R1 3.35 mm to (172.4, 81.2)
- moved U1 1.45 mm to (175.7, 80.2), turned to 180 degrees
- moved BT1 1.26 mm to (180.8, 87.2)
- moved J2 1.03 mm to (195.0, 87.2)
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Connections:
- U3 pad 21: (no net) -> GND
Routing:
- net GND: track 13.7 -> 29.3 mm, vias 11 -> 27
- net /SWCLK: track 16.6 -> 2.71 mm
- net /NRF_PWR: track 0.00 -> 13.6 mm
- net /SWDIO: track 17.2 -> 3.66 mm
- net /I2C_SDA: track 0.00 -> 8.02 mm, vias 0 -> 2
- net VCC: track 7.32 -> 14.4 mm, vias 2 -> 7
- net +VSW: track 4.69 -> 10.9 mm, vias 1 -> 5
- net /I2C_SCL: track 0.00 -> 5.94 mm
- net /NRST: track 9.30 -> 5.17 mm
- net Net-(Q1-Pad3): track 0.00 -> 1.13 mm
- net Net-(C16-Pad1): track 6.48 -> 5.50 mm
- net /SPI_MOSI: track 3.75 -> 4.40 mm
- net /SPI_MISO: track 4.99 -> 5.54 mm
- added copper zone on F.Cu, net GND
Other:
- net class Default: clearance 0.15 -> 0.2; trace_width 0.15 -> 0.1524; via_dia 0.8 -> 0.6; via_drill 0.4 -> 0.3
- rule trace_clearance: 0.15 -> 0.2
- rule trace_min: 0.1 -> 0.152

Commit message: Layout
Parts:
- added BT1: CR2032, Battery:BatteryHolder_Keystone_1060_1x2032, B.Cu at (180.8, 87.2)
- added FB1: 100 @ 100MHz, Inductor_SMD:L_0402_1005Metric, F.Cu at (181.9, 79.4)
- moved Q2 13.1 mm to (174.5, 98.0)
- moved C8 1.10 mm to (184.3, 79.9)
- moved C19 1.10 mm to (185.9, 79.9)
- moved R5 1.10 mm to (183.0, 79.4)
- moved R8 0.83 mm to (174.0, 94.2)
- moved R9 0.83 mm to (175.0, 94.2)
- moved J2 0.75 mm to (194.2, 87.2)
- moved LD1 0.18 mm to (179.2, 91.0)
- moved R7 0.15 mm to (179.2, 93.1)
Connections:
- Q1 pad 3: Net-(Q1-Pad3) -> Net-(FB1-Pad2)
- R5 pad 2: Net-(Q1-Pad3) -> Net-(FB1-Pad1)
- U2 pad 3: Net-(U2-Pad3) -> /BAT_LEVEL
- U2 pad 6: /LED_STATUS -> Net-(U2-Pad6)
- U2 pad 7: /BAT_LEVEL -> /LED_STATUS
- U3 pad 21: GND -> (no net)
Routing:
- net /SWDIO: track 3.66 -> 27.1 mm
- net /SWCLK: track 2.71 -> 24.5 mm
- net Net-(BT1-Pad1): track 0.00 -> 11.3 mm, vias 0 -> 2
- net GND: track 29.3 -> 36.0 mm, vias 27 -> 64
- net VCC: track 14.4 -> 20.7 mm, vias 7 -> 11
- net /NRST: track 5.17 -> 10.7 mm
- net /BAT_LEVEL: track 0.00 -> 5.33 mm
- net +VSW: track 10.9 -> 14.6 mm, vias 5 -> 8
- net /LED_STATUS: track 0.00 -> 2.78 mm
- net Net-(LD1-Pad1): track 0.00 -> 1.13 mm
- net Net-(Q1-Pad3): track 1.13 -> 0.00 mm
- net Net-(FB1-Pad2): track 0.00 -> 1.13 mm
- net Net-(FB1-Pad1): track 0.00 -> 1.10 mm
- added copper zone on B.Cu, net GND
Other:
- board size 35.9 x 36.4 mm -> 33.5 x 34 mm

Commit message: Layout
Parts:
- removed the BT1 at (180.8, 87.2)
- added G***: LOGO, ak:lemonhead, B.Cu at (168.8, 83.5)
- added G***: LOGO, ak:LN-10x5mm, F.Cu at (189.0, 96.5)
- moved C13 1.00 mm to (188.2, 89.2)
- moved C15 1.00 mm to (188.2, 90.2)
- moved R6 0.25 mm to (185.1, 83.5)
- moved C18 0.05 mm to (181.8, 90.5)
Connections:
- J1 pad 6: Net-(J1-Pad6) -> (no net)
- J1 pad 7: Net-(J1-Pad7) -> (no net)
- J1 pad 8: Net-(J1-Pad8) -> (no net)
- U1 pad 3: Net-(U1-Pad3) -> (no net)
- U1 pad 4: Net-(U1-Pad4) -> (no net)
- U1 pad 7: GND -> /TEMP
- U2 pad 10: Net-(U2-Pad10) -> (no net)
- U2 pad 2: Net-(U2-Pad2) -> (no net)
- U2 pad 23: Net-(U2-Pad23) -> (no net)
- U2 pad 24: Net-(U2-Pad24) -> (no net)
- U2 pad 25: Net-(U2-Pad25) -> (no net)
- U2 pad 26: Net-(U2-Pad26) -> (no net)
- U2 pad 6: Net-(U2-Pad6) -> (no net)
- U2 pad 9: Net-(U2-Pad9) -> (no net)
Routing:
- net /SWDIO: track 27.1 -> 26.0 mm
- net VCC: track 20.7 -> 21.6 mm
- net /SWCLK: track 24.5 -> 23.9 mm
- net GND: track 36.0 -> 36.6 mm, vias 64 -> 120
- added copper zone on F.Cu, net /TEMP
Other:
- board text added: "Made by Lemonhead"
- board text added: "NinjaRF24"
- board text added: "Rev. A 10/2020"

Commit message: Finalizing
Parts:
- FB1: footprint Inductor_SMD:L_0402_1005Metric -> Inductor_SMD:L_0805_2012Metric
- LD1: footprint LED_SMD:LED_0402_1005Metric -> LED_SMD:LED_0603_1608Metric
- moved C19 1.60 mm to (187.5, 79.9)
- moved C8 1.45 mm to (185.8, 79.9)
- moved R5 1.26 mm to (184.2, 79.2)
- moved R7 0.96 mm to (179.4, 94.0)
- moved FB1 0.62 mm to (182.5, 79.2)
- moved LD1 0.43 mm to (179.4, 91.4)
Connections:
- U3 pad 21: (no net) -> GND
Routing:
- net +VSW: track 14.6 -> 17.1 mm, vias 8 -> 6
- net GND: track 36.6 -> 34.6 mm, vias 120 -> 118
- net Net-(FB1-Pad2): track 1.13 -> 2.34 mm
- net Net-(FB1-Pad1): track 1.10 -> 1.94 mm

Commit message: Minor changes
Parts:
- added Q3: AO3401A, Package_TO_SOT_SMD:SOT-23, F.Cu at (169.8, 90.8)
- added R11: 1M, Resistor_SMD:R_0402_1005Metric, F.Cu at (170.2, 88.5)
- added R12: 680, Resistor_SMD:R_0402_1005Metric, F.Cu at (178.5, 94.2)
- added REF**: JLCPCB Tooling Hole, ak:JLCPCB Tooling Hole, F.Cu at (191.5, 98.5)
- added REF**: JLCPCB Tooling Hole, ak:JLCPCB Tooling Hole, F.Cu at (191.5, 76.0)
- added REF**: JLCPCB Tooling Hole, ak:JLCPCB Tooling Hole, F.Cu at (170.0, 76.0)
- C12, C14: value 22pF -> 10pF
- C19, C8: value TBD -> 22uF
- FB1: value 100 @ 100MHz -> 100Ohm@100MHz
- J2: footprint Connector_Coaxial:SMA_Samtec_SMA-J-P-H-ST-EM1_EdgeMount -> ak:SMA_Samtec_SMA-J-P-H-ST-EM1_EdgeMount
- Q1, Q2: value NTK3139P -> AO3401A; footprint Package_TO_SOT_SMD:SOT-723 -> Package_TO_SOT_SMD:SOT-23
- R5: value TBD -> 1k
- R8, R9: value TBD -> 680
- U1: value Si7021-A20 -> SHT21
- moved R7 8.40 mm to (171.0, 94.0), turned to 90 degrees
- moved R2 7.10 mm to (171.4, 82.2), turned to 0 degrees
- moved LD1 6.78 mm to (173.2, 94.2), turned to 0 degrees
- moved R9 4.50 mm to (179.5, 94.2)
- moved R8 3.50 mm to (177.5, 94.2)
- moved R4 2.10 mm to (179.0, 77.3), turned to 270 degrees
- moved C2 1.05 mm to (175.8, 94.2), turned to 90 degrees
- moved G*** 1.03 mm to (188.8, 95.5)
- moved C3 1.00 mm to (171.9, 79.7)
- moved R1 1.00 mm to (171.4, 81.2)
- moved U1 1.00 mm to (174.7, 80.2)
- moved FB1 1.00 mm to (182.8, 80.2)
- moved Q1 0.89 mm to (180.0, 80.2)
- moved J2 0.75 mm to (195.0, 87.2)
- moved Q2 0.60 mm to (175.1, 98.0)
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Connections:
- J1 pad 6: (no net) -> Net-(J1-Pad6)
- J1 pad 7: (no net) -> Net-(J1-Pad7)
- J1 pad 8: (no net) -> Net-(J1-Pad8)
- R8 pad 1: VCC -> Net-(Q3-Pad3)
- U1 pad 3: (no net) -> Net-(U1-Pad3)
- U1 pad 4: (no net) -> Net-(U1-Pad4)
- U2 pad 10: (no net) -> Net-(U2-Pad10)
- U2 pad 2: (no net) -> Net-(U2-Pad2)
- U2 pad 23: (no net) -> /BAT_CHECK
- U2 pad 24: (no net) -> Net-(U2-Pad24)
- U2 pad 25: (no net) -> Net-(U2-Pad25)
- U2 pad 26: (no net) -> Net-(U2-Pad26)
- U2 pad 3: /BAT_LEVEL -> /LED_STATUS
- U2 pad 6: (no net) -> Net-(U2-Pad6)
- U2 pad 7: /LED_STATUS -> /BAT_LEVEL
- U2 pad 9: (no net) -> Net-(U2-Pad9)
Routing:
- net Net-(Q3-Pad3): track 0.00 -> 11.4 mm
- net +VSW: track 17.1 -> 8.78 mm
- net /BAT_CHECK: track 0.00 -> 6.09 mm
- net /SWCLK: track 23.9 -> 27.9 mm
- net /SWDIO: track 26.0 -> 30.0 mm
- net Net-(BT1-Pad1): track 11.3 -> 7.76 mm
- net GND: track 34.6 -> 31.2 mm, vias 118 -> 112
- net /BAT_LEVEL: track 5.33 -> 7.99 mm
- net VCC: track 21.6 -> 19.1 mm, vias 11 -> 14
- net /LED_STATUS: track 2.97 -> 5.46 mm
- net /NRF_PWR: track 13.5 -> 12.9 mm
- net /NRST: vias 0 -> 2
- added copper zone on F.Cu, net Net-(BT1-Pad1)
- added copper zone on F.Cu, net VCC
- removed copper zone on F.Cu, net /TEMP
Other:
- board text added: "JLCJLCJLCJLC"

Commit message: Minor changes
Parts:
- added C20: 100uF, Capacitor_Tantalum_SMD:CP_EIA-3528-15_AVX-H, F.Cu at (182.5, 76.5)
- U1: value SHT21 -> SI7021
- moved C3 5.55 mm to (176.8, 77.0), turned to 270 degrees
- moved R1 4.12 mm to (175.5, 81.8), turned to 180 degrees
- moved U1 3.76 mm to (174.0, 76.5), turned to 0 degrees
- moved R4 3.20 mm to (177.8, 80.2), turned to 90 degrees
- moved R2 2.16 mm to (173.5, 81.8)
- moved Q1 0.75 mm to (180.0, 81.0)
Routing:
- net /I2C_SCL: track 6.17 -> 14.6 mm
- net /I2C_SDA: track 8.55 -> 13.2 mm, vias 2 -> 0
- net /NRF_PWR: track 12.9 -> 9.26 mm
- net VCC: track 19.1 -> 21.7 mm, vias 14 -> 13
- net +VSW: track 8.78 -> 6.44 mm, vias 6 -> 7
- net Net-(FB1-Pad2): track 2.48 -> 3.23 mm
- net GND: track 31.2 -> 31.4 mm, vias 112 -> 114
- added copper zone on F.Cu, net +VSW
Other:
- board text added: "+"
