File: NRF24.sch (KiCad schematic (older format))
At the start: 28 parts

Commit message: Rough component placement
Parts:
- removed U?: STM32L031G6UxS, Package_DFN_QFN:QFN-28_4x4mm_P0.5mm, symbol MCU_ST_STM32L0:STM32L031G6UxS
- added C1: 10uF, Capacitor_SMD:C_0603_1608Metric, symbol Device:C_Small
- added C2, C4, C5, C6: 100nF, Capacitor_SMD:C_0402_1005Metric, symbol Device:C_Small
- added C7: 1uF, Capacitor_SMD:C_0603_1608Metric, symbol Device:C_Small
- added LD1: GREEN, LED_SMD:LED_0603_1608Metric, symbol Device:LED_Small
- added Q2: PMF170XP, Package_TO_SOT_SMD:SOT-323_SC-70, symbol Device:Q_PMOS_GSD
- added R3: 0R, Resistor_SMD:R_0402_1005Metric, symbol Device:R_Small
- added R7: 2k2, Resistor_SMD:R_0603_1608Metric, symbol Device:R_Small
- added R8, R9: TBD, Resistor_SMD:R_0402_1005Metric, symbol Device:R_Small
- added U2: STM32L031G6Ux, Package_DFN_QFN:QFN-28_4x4mm_P0.5mm, symbol MCU_ST_STM32L0:STM32L031G6Ux
- BT1: renamed from BT?; footprint (none) -> Battery:BatteryHolder_Keystone_1060_1x2032
- C10, C11, C12, C13, C14, C15, C16, C17, C3, C9: renamed from C?; footprint (none) -> Capacitor_SMD:C_0402_1005Metric
- C8: renamed from C?; footprint (none) -> Capacitor_SMD:C_0603_1608Metric
- J1: renamed from J?; footprint (none) -> Connector_PinHeader_1.27mm:PinHeader_2x05_P1.27mm_Vertical_SMD
- J2: renamed from J?; footprint (none) -> Connector_Coaxial:SMA_Samtec_SMA-J-P-H-ST-EM1_EdgeMount
- L2, L3, L4: renamed from L?; footprint (none) -> Inductor_SMD:L_0402_1005Metric
- Q1: renamed from Q?; value NX3008PBKW -> PMF170XP; footprint (none) -> Package_TO_SOT_SMD:SOT-323_SC-70
- R1, R10, R2, R4, R5, R6: renamed from R?; footprint (none) -> Resistor_SMD:R_0402_1005Metric
- Y1: renamed from Y?; footprint (none) -> Crystal:Crystal_SMD_3225-4Pin_3.2x2.5mm
- gave numbers to parts that had none: 2
Connections:
- net labels added: BAT_LEVEL, BOOT0, I2C_SCL, I2C_SDA, LED_STATUS, NRF_CE, NRF_IRQ, NRF_PWR, NRST, SPI_CSN, SPI_MISO, SPI_MOSI, SPI_SCK, SWCLK, SWDIO, VCC
- net labels removed: +BATT, SCL, SDA
- wire segments 133 -> 196
- no-connect marks 1 -> 10
Other:
- moved on the sheet: BT1, C10, C11, C12, C13, C14, C15, C16, C17, C3, C8, C9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

Commit message: Layout
Parts:
- added C18: 10nF, Capacitor_SMD:C_0402_1005Metric, symbol Device:C_Small
Connections:
- net GND: now also C18.1
- net NRF_CE: now also U2.15 (PB1); no longer U2.8 (PA2)
- net NRF_IRQ: now also U2.8 (PA2); no longer U2.9 (PA3)
- net NRF_PWR: now also U2.18 (PA8); no longer U2.14 (PB0)
- net +VSW: now reaches C11.2, C8.1, C9.2, R5.1, U3.15 (VDD), U3.18 (VDD), U3.7 (VDD)
- net +VSW: now also C18.2
- net SPI_CSN: no longer names the net of U2.10 (PA4)
- net SPI_CSN: no longer U3.2 (CSN)
- new net NRF_CSN: U2.14 (PB0), U3.2 (CSN)
- no-connect marks 10 -> 8
Other:
- moved on the sheet: C8, Q1, R4, R5
Changed lines of the file:
@@
 L Device:Q_PMOS_GSD Q1
 U 1 1 5F6E35A8
-P 6200 1150
-F 0 "Q1" V 6542 1150 50  0000 C CNN
-F 1 "PMF170XP" V 6451 1150 50  0000 C CNN
-F 2 "Package_TO_SOT_SMD:SOT-323_SC-70" H 6400 1250 50  0001 C CNN
-F 3 "~" H 6200 1150 50  0001 C CNN
-	1    6200 1150
+P 5750 1150
+F 0 "Q1" V 6092 1150 50  0000 C CNN
+F 1 "PMF170XP" V 6001 1150 50  0000 C CNN
+F 2 "Package_TO_SOT_SMD:SOT-323_SC-70" H 5950 1250 50  0001 C CNN
+F 3 "~" H 5750 1150 50  0001 C CNN
+	1    5750 1150
 	0    1    -1   0
 $EndComp
@@
 L Device:R_Small R5
 U 1 1 5F6EDFC5
-P 6650 1050
-F 0 "R5" V 6600 1200 50  0000 C CNN
-F 1 "TBD" V 6600 900 50  0000 C CNN
-F 2 "Resistor_SMD:R_0402_1005Metric" H 6650 1050 50  0001 C CNN
-F 3 "~" H 6650 1050 50  0001 C CNN
-	1    6650 1050
+P 6200 1050
+F 0 "R5" V 6150 1200 50  0000 C CNN
+F 1 "TBD" V 6150 900 50  0000 C CNN
+F 2 "Resistor_SMD:R_0402_1005Metric" H 6200 1050 50  0001 C CNN
+F 3 "~" H 6200 1050 50  0001 C CNN
+	1    6200 1050
 	0    1    1    0
 $EndComp
 Wire Wire Line
-	6400 1050 6550 1050
+	5950 1050 6100 1050
 Wire Wire Line
 	8150 1050 8250 1050
@@
 L Device:R_Small R4
 U 1 1 5F6FC380
-P 5800 1250
-F 0 "R4" H 5859 1296 50  0000 L CNN
-F 1 "1M" H 5859 1205 50  0000 L CNN
-F 2 "Resistor_SMD:R_0402_1005Metric" H 5800 1250 50  0001 C CNN
-F 3 "~" H 5800 1250 50  0001 C CNN
-	1    5800 1250
-	1    0    0    -1
-$EndComp
-Wire Wire Line
-	5800 1150 5800 1050
-Wire Wire Line
-	5800 1050 6000 1050
-Wire Wire Line
-	5800 1350 5800 1450
-Wire Wire Line
-	6200 1450 6200 1350
+P 5350 1250
+F 0 "R4" H 5409 1296 50  0000 L CNN
+F 1 "1M" H 5409 1205 50  0000 L CNN
+F 2 "Resistor_SMD:R_0402_1005Metric" H 5350 1250 50  0001 C CNN
+F 3 "~" H 5350 1250 50  0001 C CNN
+	1    5350 1250
+	1    0    0    -1
+$EndComp
+Wire Wire Line
+	5350 1150 5350 1050
+Wire Wire Line
+	5350 1050 5550 1050
+Wire Wire Line
+	5350 1350 5350 1450
+Wire Wire Line
+	5750 1450 5750 1350
 Wire Wire Line
 	5000 4550 5100 4550
@@
 	5000 4550 5000 4600
 Wire Wire Line
-	5800 1450 6200 1450
+	5350 1450 5750 1450
 Wire Wire Line
 	1900 4800 2350 4800
@@
 	1350 5750 1400 5750
 Wire Wire Line
-	5800 950  5800 1050
-Connection ~ 5800 1050
-Connection ~ 6900 1050
-Wire Wire Line
-	6900 1050 7250 1050
+	5350 950  5350 1050
+Connection ~ 5350 1050
+Connection ~ 6450 1050
+Wire Wire Line
+	6450 1050 6650 1050
 Wire Wire Line
 	7250 1050 7250 1100
@@
 L power:GND #PWR017
 U 1 1 5F6F9C7B
-P 6900 1300
-F 0 "#PWR017" H 6900 1050 50  0001 C CNN
-F 1 "GND" H 6905 1127 50  0001 C CNN
-F 2 "" H 6900 1300 50  0001 C CNN
-F 3 "" H 6900 1300 50  0001 C CNN
-	1    6900 1300
-	1    0    0    -1
-$EndComp
-Wire Wire Line
-	6900 1050 6900 1100
-Wire Wire Line
-	6750 1050 6900 1050
+P 6450 1300
+F 0 "#PWR017" H 6450 1050 50  0001 C CNN
+F 1 "GND" H 6455 1127 50  0001 C CNN
+F 2 "" H 6450 1300 50  0001 C CNN
+F 3 "" H 6450 1300 50  0001 C CNN
+	1    6450 1300
+	1    0    0    -1
+$EndComp
+Wire Wire Line
+	6450 1050 6450 1100
+Wire Wire Line
+	6300 1050 6450 1050
 $Comp
 L Device:C_Small C8
 U 1 1 5F6EEBBB
-P 6900 1200
-F 0 "C8" H 6992 1246 50  0000 L CNN
-F 1 "TBD" H 6992 1155 50  0000 L CNN
-F 2 "Capacitor_SMD:C_0603_1608Metric" H 6900 1200 50  0001 C CNN
-F 3 "~" H 6900 1200 50  0001 C CNN
-	1    6900 1200
+P 6450 1200
+F 0 "C8" H 6542 1246 50  0000 L CNN
+F 1 "TBD" H 6542 1155 50  0000 L CNN
+F 2 "Capacitor_SMD:C_0603_1608Metric" H 6450 1200 50  0001 C CNN
+F 3 "~" H 6450 1200 50  0001 C CNN
+	1    6450 1200
 	1    0    0    -1
 $EndComp
@@
 $EndComp
 Wire Wire Line
-	5800 1450 5350 1450
-Connection ~ 5800 1450
+	5350 1450 4900 1450
+Connection ~ 5350 1450
 Connection ~ 4100 950
 Wire Wire Line
@@
 SPI_MOSI
 Text Label 7200 1800 0    50   ~ 0
-SPI_CSN
+NRF_CSN
 Text Label 2200 1500 0    50   ~ 0
 I2C_SCL
@@
 Wire Wire Line
 	7800 5800 7800 5850
-Text Label 5350 1450 0    50   ~ 0
+Text Label 4900 1450 0    50   ~ 0
 NRF_PWR
 Wire Wire Line
@@
 Text Label 7350 5500 0    50   ~ 0
 LED_STATUS
-Text Label 6150 5200 2    50   ~ 0
-SPI_CSN
 Text Label 7200 2000 0    50   ~ 0
 NRF_CE
@@
 Text Label 8300 5800 0    50   ~ 0
 BAT_LEVEL
-NoConn ~ 4500 5400
 NoConn ~ 4500 5500
-NoConn ~ 4500 5800
 NoConn ~ 4500 5900
 NoConn ~ 4500 6000
 NoConn ~ 4500 6100
 NoConn ~ 5600 6100
-NoConn ~ 5600 5600
 $Comp
 L power:GND #PWR0101
@@
 	8350 950  8350 1050
 Connection ~ 8350 1050
+Text Label 3950 5800 0    50   ~ 0
+NRF_CE
 Text Label 6150 5000 2    50   ~ 0
-NRF_CE
-Text Label 6150 5100 2    50   ~ 0
 NRF_IRQ
 Wire Wire Line
@@
 Wire Wire Line
 	5600 5100 6150 5100
-Text Label 3950 5700 0    50   ~ 0
+Text Label 6150 5600 2    50   ~ 0
 NRF_PWR
 $Comp
@@
 L power:VCC #PWR016
 U 1 1 5F79FBFF
-P 5800 950
-F 0 "#PWR016" H 5800 800 50  0001 C CNN
-F 1 "VCC" H 5815 1123 50  0000 C CNN
-F 2 "" H 5800 950 50  0001 C CNN
-F 3 "" H 5800 950 50  0001 C CNN
-	1    5800 950
+P 5350 950
+F 0 "#PWR016" H 5350 800 50  0001 C CNN
+F 1 "VCC" H 5365 1123 50  0000 C CNN
+F 2 "" H 5350 950 50  0001 C CNN
+F 3 "" H 5350 950 50  0001 C CNN
+	1    5350 950
 	1    0    0    -1
 $EndComp
@@
 	1    0    0    -1
 $EndComp
+Text Label 3950 5700 0    50   ~ 0
+NRF_CSN
+NoConn ~ 4500 5400
+Wire Wire Line
+	4500 5800 3950 5800
+Wire Wire Line
+	5600 5600 6150 5600
+$Comp
+L Device:C_Small C18
+U 1 1 5F77A80D
+P 6900 1200
+F 0 "C18" H 6808 1154 50  0000 R CNN
+F 1 "10nF" H 6808 1245 50  0000 R CNN
+F 2 "Capacitor_SMD:C_0402_1005Metric" H 6900 1200 50  0001 C CNN
+F 3 "~" H 6900 1200 50  0001 C CNN
+	1    6900 1200
+	-1   0    0    1
+$EndComp
+Wire Wire Line
+	6900 1050 6900 1100
+Connection ~ 6900 1050
+Wire Wire Line
+	6900 1050 7250 1050
+$Comp
+L power:GND #PWR0102
+U 1 1 5F787AC1
+P 6900 1300
+F 0 "#PWR0102" H 6900 1050 50  0001 C CNN
+F 1 "GND" H 6905 1127 50  0001 C CNN
+F 2 "" H 6900 1300 50  0001 C CNN
+F 3 "" H 6900 1300 50  0001 C CNN
+	1    6900 1300
+	1    0    0    -1
+$EndComp
+$Comp
+L power:+VSW #PWR?
+U 1 1 5F79F380
+P 6650 950
+F 0 "#PWR?" H 6650 800 50  0001 C CNN
+F 1 "+VSW" H 6665 1123 50  0000 C CNN
+F 2 "" H 6650 950 50  0001 C CNN
+F 3 "" H 6650 950 50  0001 C CNN
+	1    6650 950
+	1    0    0    -1
+$EndComp
+Wire Wire Line
+	6650 950  6650 1050
+Connection ~ 6650 1050
+Wire Wire Line
+	6650 1050 6900 1050
 $EndSCHEMATC

Commit message: Layout
Parts:
- added C19: TBD, Capacitor_SMD:C_0603_1608Metric, symbol Device:C_Small
- LD1: value GREEN -> BLUE; footprint LED_SMD:LED_0603_1608Metric -> LED_SMD:LED_0402_1005Metric
- Q1, Q2: value PMF170XP -> NTK3139P; footprint Package_TO_SOT_SMD:SOT-323_SC-70 -> Package_TO_SOT_SMD:SOT-723
- R7: value 2k2 -> 10R; footprint Resistor_SMD:R_0603_1608Metric -> Resistor_SMD:R_0402_1005Metric
Connections:
- net +VSW: now also C19.1
- net GND: now also C19.2
Other:
- moved on the sheet: Q1, R4, R5
Changed lines of the file:
@@
 L Device:Q_PMOS_GSD Q1
 U 1 1 5F6E35A8
-P 5750 1150
-F 0 "Q1" V 6092 1150 50  0000 C CNN
-F 1 "PMF170XP" V 6001 1150 50  0000 C CNN
-F 2 "Package_TO_SOT_SMD:SOT-323_SC-70" H 5950 1250 50  0001 C CNN
-F 3 "~" H 5750 1150 50  0001 C CNN
-	1    5750 1150
+P 5450 1150
+F 0 "Q1" V 5792 1150 50  0000 C CNN
+F 1 "NTK3139P" V 5701 1150 50  0000 C CNN
+F 2 "Package_TO_SOT_SMD:SOT-723" H 5650 1250 50  0001 C CNN
+F 3 "~" H 5450 1150 50  0001 C CNN
+	1    5450 1150
 	0    1    -1   0
 $EndComp
@@
 L Device:R_Small R5
 U 1 1 5F6EDFC5
-P 6200 1050
-F 0 "R5" V 6150 1200 50  0000 C CNN
-F 1 "TBD" V 6150 900 50  0000 C CNN
-F 2 "Resistor_SMD:R_0402_1005Metric" H 6200 1050 50  0001 C CNN
-F 3 "~" H 6200 1050 50  0001 C CNN
-	1    6200 1050
+P 5900 1050
+F 0 "R5" V 5850 1200 50  0000 C CNN
+F 1 "TBD" V 5850 900 50  0000 C CNN
+F 2 "Resistor_SMD:R_0402_1005Metric" H 5900 1050 50  0001 C CNN
+F 3 "~" H 5900 1050 50  0001 C CNN
+	1    5900 1050
 	0    1    1    0
 $EndComp
 Wire Wire Line
-	5950 1050 6100 1050
+	5650 1050 5800 1050
 Wire Wire Line
 	8150 1050 8250 1050
@@
 L Device:R_Small R4
 U 1 1 5F6FC380
-P 5350 1250
-F 0 "R4" H 5409 1296 50  0000 L CNN
-F 1 "1M" H 5409 1205 50  0000 L CNN
-F 2 "Resistor_SMD:R_0402_1005Metric" H 5350 1250 50  0001 C CNN
-F 3 "~" H 5350 1250 50  0001 C CNN
-	1    5350 1250
-	1    0    0    -1
-$EndComp
-Wire Wire Line
-	5350 1150 5350 1050
-Wire Wire Line
-	5350 1050 5550 1050
-Wire Wire Line
-	5350 1350 5350 1450
-Wire Wire Line
-	5750 1450 5750 1350
+P 5050 1250
+F 0 "R4" H 5109 1296 50  0000 L CNN
+F 1 "1M" H 5109 1205 50  0000 L CNN
+F 2 "Resistor_SMD:R_0402_1005Metric" H 5050 1250 50  0001 C CNN
+F 3 "~" H 5050 1250 50  0001 C CNN
+	1    5050 1250
+	1    0    0    -1
+$EndComp
+Wire Wire Line
+	5050 1150 5050 1050
+Wire Wire Line
+	5050 1050 5250 1050
+Wire Wire Line
+	5050 1350 5050 1450
+Wire Wire Line
+	5450 1450 5450 1350
 Wire Wire Line
 	5000 4550 5100 4550
@@
 	5000 4550 5000 4600
 Wire Wire Line
-	5350 1450 5750 1450
+	5050 1450 5450 1450
 Wire Wire Line
 	1900 4800 2350 4800
@@
 	1350 5750 1400 5750
 Wire Wire Line
-	5350 950  5350 1050
-Connection ~ 5350 1050
+	5050 950  5050 1050
+Connection ~ 5050 1050
 Connection ~ 6450 1050
 Wire Wire Line
@@
 	6450 1050 6450 1100
 Wire Wire Line
-	6300 1050 6450 1050
+	6000 1050 6150 1050
 $Comp
 L Device:C_Small C8
@@
 $EndComp
 Wire Wire Line
-	5350 1450 4900 1450
-Connection ~ 5350 1450
+	5050 1450 4600 1450
+Connection ~ 5050 1450
 Connection ~ 4100 950
 Wire Wire Line
@@
 P 7800 5700
 F 0 "LD1" V 7846 5630 50  0000 R CNN
-F 1 "GREEN" V 7755 5630 50  0000 R CNN
-F 2 "LED_SMD:LED_0603_1608Metric" V 7800 5700 50  0001 C CNN
+F 1 "BLUE" V 7755 5630 50  0000 R CNN
+F 2 "LED_SMD:LED_0402_1005Metric" V 7800 5700 50  0001 C CNN
 F 3 "~" V 7800 5700 50  0001 C CNN
 	1    7800 5700
@@
 P 7800 5950
 F 0 "R7" H 7859 5996 50  0000 L CNN
-F 1 "2k2" H 7859 5905 50  0000 L CNN
-F 2 "Resistor_SMD:R_0603_1608Metric" H 7800 5950 50  0001 C CNN
+F 1 "10R" H 7859 5905 50  0000 L CNN
+F 2 "Resistor_SMD:R_0402_1005Metric" H 7800 5950 50  0001 C CNN
 F 3 "~" H 7800 5950 50  0001 C CNN
 	1    7800 5950
@@
 Wire Wire Line
 	7800 5800 7800 5850
-Text Label 4900 1450 0    50   ~ 0
+Text Label 4600 1450 0    50   ~ 0
 NRF_PWR
 Wire Wire Line
@@
 P 1450 1150
 F 0 "Q2" V 1792 1150 50  0000 C CNN
-F 1 "PMF170XP" V 1701 1150 50  0000 C CNN
-F 2 "Package_TO_SOT_SMD:SOT-323_SC-70" H 1650 1250 50  0001 C CNN
+F 1 "NTK3139P" V 1701 1150 50  0000 C CNN
+F 2 "Package_TO_SOT_SMD:SOT-723" H 1650 1250 50  0001 C CNN
 F 3 "~" H 1450 1150 50  0001 C CNN
 	1    1450 1150
@@
 L power:VCC #PWR016
 U 1 1 5F79FBFF
-P 5350 950
-F 0 "#PWR016" H 5350 800 50  0001 C CNN
-F 1 "VCC" H 5365 1123 50  0000 C CNN
-F 2 "" H 5350 950 50  0001 C CNN
-F 3 "" H 5350 950 50  0001 C CNN
-	1    5350 950
+P 5050 950
+F 0 "#PWR016" H 5050 800 50  0001 C CNN
+F 1 "VCC" H 5065 1123 50  0000 C CNN
+F 2 "" H 5050 950 50  0001 C CNN
+F 3 "" H 5050 950 50  0001 C CNN
+	1    5050 950
 	1    0    0    -1
 $EndComp
@@
 $EndComp
 $Comp
-L power:+VSW #PWR?
+L power:+VSW #PWR0103
 U 1 1 5F79F380
 P 6650 950
-F 0 "#PWR?" H 6650 800 50  0001 C CNN
+F 0 "#PWR0103" H 6650 800 50  0001 C CNN
 F 1 "+VSW" H 6665 1123 50  0000 C CNN
 F 2 "" H 6650 950 50  0001 C CNN
@@
 Wire Wire Line
 	6650 1050 6900 1050
+$Comp
+L Device:C_Small C19
+U 1 1 5F7546E4
+P 6150 1200
+F 0 "C19" H 6242 1246 50  0000 L CNN
+F 1 "TBD" H 6242 1155 50  0000 L CNN
+F 2 "Capacitor_SMD:C_0603_1608Metric" H 6150 1200 50  0001 C CNN
+F 3 "~" H 6150 1200 50  0001 C CNN
+	1    6150 1200
+	1    0    0    -1
+$EndComp
+Wire Wire Line
+	6150 1100 6150 1050
+Connection ~ 6150 1050
+Wire Wire Line
+	6150 1050 6450 1050
+$Comp
+L power:GND #PWR01
+U 1 1 5F760EE7
+P 6150 1300
+F 0 "#PWR01" H 6150 1050 50  0001 C CNN
+F 1 "GND" H 6155 1127 50  0001 C CNN
+F 2 "" H 6150 1300 50  0001 C CNN
+F 3 "" H 6150 1300 50  0001 C CNN
+	1    6150 1300
+	1    0    0    -1
+$EndComp
 $EndSCHEMATC

Commit message: Layout
Parts:
- added FB1: 100 @ 100MHz, Inductor_SMD:L_0402_1005Metric, symbol Device:Ferrite_Bead_Small
Connections:
- net BAT_LEVEL: now also U2.3 (PC15); no longer U2.7 (PA1)
- net LED_STATUS: now also U2.7 (PA1); no longer U2.6 (PA0)
- net at Q1.3 (D): now also FB1.2; no longer R5.2
- new net: FB1.1, R5.2
- no-connect marks 8 -> 10
Other:
- moved on the sheet: C3, Q1, R1, R2, R4, U1

Commit message: Layout
Connections:
- net GND: no longer U1.7 (PAD)
- new net TEMP: U1.7 (PAD)
- no-connect marks 10 -> 11
Changed lines of the file:
@@
 L power:GND #PWR06
 U 1 1 5F6F7763
-P 2300 3250
-F 0 "#PWR06" H 2300 3000 50  0001 C CNN
-F 1 "GND" H 2305 3077 50  0001 C CNN
-F 2 "" H 2300 3250 50  0001 C CNN
-F 3 "" H 2300 3250 50  0001 C CNN
-	1    2300 3250
+P 2200 3200
+F 0 "#PWR06" H 2200 2950 50  0001 C CNN
+F 1 "GND" H 2205 3027 50  0001 C CNN
+F 2 "" H 2200 3200 50  0001 C CNN
+F 3 "" H 2200 3200 50  0001 C CNN
+	1    2200 3200
 	1    0    0    -1
 $EndComp
@@
 Wire Wire Line
 	2900 2400 2900 2500
-Wire Wire Line
-	2200 3150 2200 3200
-Wire Wire Line
-	2200 3200 2300 3200
-Wire Wire Line
-	2400 3200 2400 3150
-Wire Wire Line
-	2300 3250 2300 3200
-Connection ~ 2300 3200
-Wire Wire Line
-	2300 3200 2400 3200
 Wire Wire Line
 	1350 5800 1350 5750
@@
 	1    0    0    -1
 $EndComp
+Wire Wire Line
+	2200 3150 2200 3200
+Wire Wire Line
+	2400 3300 2650 3300
+Wire Wire Line
+	2400 3150 2400 3300
+Text Label 2650 3300 2    50   ~ 0
+TEMP
+NoConn ~ 2650 3300
 $EndSCHEMATC
