File: NRF24.sch (KiCad schematic (older format))
At the start: 43 parts, among them J1 Conn_ARM_JTAG_SWD_10, J2 SMA, Q1 NTK3139P, Q2 NTK3139P, U1 Si7021-A20, U2 STM32L031G6Ux, U3 nRF24L01P, Y1 16MHz

Commit message: Finalizing
Parts:
- C1: LCSC (none) -> C19702
- C10: LCSC (none) -> C1585
- C11: LCSC (none) -> C1523
- C13: LCSC (none) -> C1531
- C15: LCSC (none) -> C1569
- C16: LCSC (none) -> C1552
- C17: LCSC (none) -> C1550
- C18, C9: LCSC (none) -> C15195
- C19, C8: value TBD -> 22uF; LCSC (none) -> C59461
- C2, C3, C4, C5, C6: LCSC (none) -> C1525
- C7: LCSC (none) -> C15849
- FB1: footprint Inductor_SMD:L_0402_1005Metric -> Inductor_SMD:L_0805_2012Metric; LCSC (none) -> C1017
- L2: LCSC (none) -> C16208
- L3: LCSC (none) -> C27123
- L4: LCSC (none) -> C14033
- LD1: footprint LED_SMD:LED_0402_1005Metric -> LED_SMD:LED_0603_1608Metric; LCSC (none) -> LED_0603
- Q1, Q2: LCSC (none) -> C415718
- R1, R2: LCSC (none) -> C25900
- R10, R4: LCSC (none) -> C26083
- R3: LCSC (none) -> C17168
- R6: LCSC (none) -> C25768
- R7: LCSC (none) -> C25077
- U1: LCSC (none) -> C132603
- U2: LCSC (none) -> C96514
- U3: LCSC (none) -> C8791
- Y1: LCSC (none) -> C13738
Changed lines of the file:
@@
 F 2 "Package_DFN_QFN:QFN-20-1EP_4x4mm_P0.5mm_EP2.5x2.5mm" H 8450 2800 50  0001 L CIN
 F 3 "http://www.nordicsemi.com/eng/content/download/2726/34069/file/nRF24L01P_Product_Specification_1_0.pdf" H 8250 2100 50  0001 C CNN
+F 4 "C8791" H 8250 2000 50  0001 C CNN "LCSC"
 	1    8250 2000
 	1    0    0    -1
@@
 F 2 "Crystal:Crystal_SMD_3225-4Pin_3.2x2.5mm" H 9300 3300 50  0001 C CNN
 F 3 "~" H 9300 3300 50  0001 C CNN
+F 4 "C13738" H 9300 3300 50  0001 C CNN "LCSC"
 	1    9300 3300
 	1    0    0    -1
@@
 F 2 "Package_TO_SOT_SMD:SOT-723" H 5050 1250 50  0001 C CNN
 F 3 "~" H 4850 1150 50  0001 C CNN
+F 4 "C415718" H 4850 1150 50  0001 C CNN "LCSC"
 	1    4850 1150
 	0    1    -1   0
@@
 F 2 "Resistor_SMD:R_0402_1005Metric" H 4450 1250 50  0001 C CNN
 F 3 "~" H 4450 1250 50  0001 C CNN
+F 4 "C26083" H 4450 1250 50  0001 C CNN "LCSC"
 	1    4450 1250
 	1    0    0    -1
@@
 F 2 "Resistor_SMD:R_0402_1005Metric" H 7200 2650 50  0001 C CNN
 F 3 "~" H 7200 2650 50  0001 C CNN
+F 4 "C25768" H 7200 2650 50  0001 C CNN "LCSC"
 	1    7200 2650
 	1    0    0    -1
@@
 F 2 "Resistor_SMD:R_0402_1005Metric" H 9300 2950 50  0001 C CNN
 F 3 "~" H 9300 2950 50  0001 C CNN
+F 4 "C26083" H 9300 2950 50  0001 C CNN "LCSC"
 	1    9300 2950
 	0    1    1    0
@@
 F 2 "Inductor_SMD:L_0402_1005Metric" H 9150 1900 50  0001 C CNN
 F 3 "~" H 9150 1900 50  0001 C CNN
+F 4 "C16208" H 9150 1900 50  0001 C CNN "LCSC"
 	1    9150 1900
 	1    0    0    -1
@@
 F 2 "Inductor_SMD:L_0402_1005Metric" H 9550 1700 50  0001 C CNN
 F 3 "~" H 9550 1700 50  0001 C CNN
+F 4 "C27123" H 9550 1700 50  0001 C CNN "LCSC"
 	1    9550 1700
 	0    -1   -1   0
@@
 F 2 "Capacitor_SMD:C_0402_1005Metric" H 10250 2300 50  0001 C CNN
 F 3 "~" H 10250 2300 50  0001 C CNN
+F 4 "C1550" H 10250 2300 50  0001 C CNN "LCSC"
 	1    10250 2300
 	-1   0    0    1
@@
 F 2 "Inductor_SMD:L_0402_1005Metric" H 9550 2100 50  0001 C CNN
 F 3 "~" H 9550 2100 50  0001 C CNN
+F 4 "C14033" H 9550 2100 50  0001 C CNN "LCSC"
 	1    9550 2100
 	0    1    1    0
@@
 F 2 "Capacitor_SMD:C_0402_1005Metric" H 9950 2100 50  0001 C CNN
 F 3 "~" H 9950 2100 50  0001 C CNN
+F 4 "C1552" H 9950 2100 50  0001 C CNN "LCSC"
 	1    9950 2100
 	0    1    1    0
@@
 F 2 "Resistor_SMD:R_0402_1005Metric" H 1700 2550 50  0001 C CNN
 F 3 "~" H 1700 2550 50  0001 C CNN
+F 4 "C25900" H 1700 2550 50  0001 C CNN "LCSC"
 	1    1700 2550
 	1    0    0    -1
@@
 F 2 "Resistor_SMD:R_0402_1005Metric" H 1400 2550 50  0001 C CNN
 F 3 "~" H 1400 2550 50  0001 C CNN
+F 4 "C25900" H 1400 2550 50  0001 C CNN "LCSC"
 	1    1400 2550
 	1    0    0    -1
@@
 F 2 "Package_DFN_QFN:DFN-6-1EP_3x3mm_P1mm_EP1.5x2.4mm" H 2300 2450 50  0001 C CNN
 F 3 "https://www.silabs.com/documents/public/data-sheets/Si7021-A20.pdf" H 2100 3150 50  0001 C CNN
+F 4 "C132603" H 2300 2850 50  0001 C CNN "LCSC"
 	1    2300 2850
 	1    0    0    -1
@@
 F 2 "Capacitor_SMD:C_0402_1005Metric" H 2900 2600 50  0001 C CNN
 F 3 "~" H 2900 2600 50  0001 C CNN
+F 4 "C1525" H 2900 2600 50  0001 C CNN "LCSC"
 	1    2900 2600
 	1    0    0    -1
@@
 F 2 "Capacitor_SMD:C_0402_1005Metric" H 7500 2650 50  0001 C CNN
 F 3 "~" H 7500 2650 50  0001 C CNN
+F 4 "C1585" H 7500 2650 50  0001 C CNN "LCSC"
 	1    7500 2650
 	-1   0    0    1
@@
 F 2 "Capacitor_SMD:C_0402_1005Metric" H 7600 1200 50  0001 C CNN
 F 3 "~" H 7600 1200 50  0001 C CNN
+F 4 "C1523" H 7600 1200 50  0001 C CNN "LCSC"
 	1    7600 1200
 	-1   0    0    1
@@
 F 2 "Capacitor_SMD:C_0402_1005Metric" H 7250 1200 50  0001 C CNN
 F 3 "~" H 7250 1200 50  0001 C CNN
+F 4 "C15195" H 7250 1200 50  0001 C CNN "LCSC"
 	1    7250 1200
 	-1   0    0    1
@@
 P 6450 1200
 F 0 "C8" H 6542 1246 50  0000 L CNN
-F 1 "TBD" H 6542 1155 50  0000 L CNN
+F 1 "22uF" H 6542 1155 50  0000 L CNN
 F 2 "Capacitor_SMD:C_0603_1608Metric" H 6450 1200 50  0001 C CNN
 F 3 "~" H 6450 1200 50  0001 C CNN
+F 4 "C59461" H 6450 1200 50  0001 C CNN "LCSC"
 	1    6450 1200
 	1    0    0    -1
@@
 F 2 "Capacitor_SMD:C_0402_1005Metric" H 9150 1250 50  0001 C CNN
 F 3 "~" H 9150 1250 50  0001 C CNN
+F 4 "C1531" H 9150 1250 50  0001 C CNN "LCSC"
 	1    9150 1250
 	-1   0    0    1
@@
 F 2 "Capacitor_SMD:C_0402_1005Metric" H 9900 1250 50  0001 C CNN
 F 3 "~" H 9900 1250 50  0001 C CNN
+F 4 "C1569" H 9900 1250 50  0001 C CNN "LCSC"
 	1    9900 1250
 	-1   0    0    1
@@
 F 2 "Capacitor_SMD:C_0402_1005Metric" H 3500 4950 50  0001 C CNN
 F 3 "~" H 3500 4950 50  0001 C CNN
+F 4 "C1525" H 3500 4950 50  0001 C CNN "LCSC"
 	1    3500 4950
 	-1   0    0    1
@@
 F 0 "LD1" V 7846 5630 50  0000 R CNN
 F 1 "BLUE" V 7755 5630 50  0000 R CNN
-F 2 "LED_SMD:LED_0402_1005Metric" V 7800 5700 50  0001 C CNN
+F 2 "LED_SMD:LED_0603_1608Metric" V 7800 5700 50  0001 C CNN
 F 3 "~" V 7800 5700 50  0001 C CNN
+F 4 "LED_0603" H 7800 5700 50  0001 C CNN "LCSC"
 	1    7800 5700
 	0    -1   -1   0
@@
 F 2 "Resistor_SMD:R_0402_1005Metric" H 7800 5950 50  0001 C CNN
 F 3 "~" H 7800 5950 50  0001 C CNN
+F 4 "C25077" H 7800 5950 50  0001 C CNN "LCSC"
 	1    7800 5950
 	1    0    0    -1
@@
 F 2 "Resistor_SMD:R_0402_1005Metric" H 3950 5150 50  0001 C CNN
 F 3 "~" H 3950 5150 50  0001 C CNN
+F 4 "C17168" H 3950 5150 50  0001 C CNN "LCSC"
 	1    3950 5150
 	1    0    0    -1
@@
 F 2 "Capacitor_SMD:C_0402_1005Metric" H 4300 4350 50  0001 C CNN
 F 3 "~" H 4300 4350 50  0001 C CNN
+F 4 "C1525" H 4300 4350 50  0001 C CNN "LCSC"
 	1    4300 4350
 	1    0    0    -1
@@
 F 2 "Capacitor_SMD:C_0402_1005Metric" H 3900 4350 50  0001 C CNN
 F 3 "~" H 3900 4350 50  0001 C CNN
+F 4 "C1525" H 3900 4350 50  0001 C CNN "LCSC"
 	1    3900 4350
 	1    0    0    -1
@@
 F 2 "Capacitor_SMD:C_0402_1005Metric" H 5500 4350 50  0001 C CNN
 F 3 "~" H 5500 4350 50  0001 C CNN
+F 4 "C1525" H 5500 4350 50  0001 C CNN "LCSC"
 	1    5500 4350
 	1    0    0    -1
@@
 F 2 "Capacitor_SMD:C_0603_1608Metric" H 3500 4350 50  0001 C CNN
 F 3 "~" H 3500 4350 50  0001 C CNN
+F 4 "C19702" H 3500 4350 50  0001 C CNN "LCSC"
 	1    3500 4350
 	1    0    0    -1
@@
 F 2 "Capacitor_SMD:C_0603_1608Metric" H 5950 4350 50  0001 C CNN
 F 3 "~" H 5950 4350 50  0001 C CNN
+F 4 "C15849" H 5950 4350 50  0001 C CNN "LCSC"
 	1    5950 4350
 	1    0    0    -1
@@
 F 2 "Package_DFN_QFN:QFN-28_4x4mm_P0.5mm" H 4600 4600 50  0001 R CNN
 F 3 "http://www.st.com/st-web-ui/static/active/en/resource/technical/document/datasheet/DM00140359.pdf" H 5100 5400 50  0001 C CNN
+F 4 "C96514" H 5100 5400 50  0001 C CNN "LCSC"
 	1    5100 5400
 	1    0    0    -1
@@
 F 2 "Package_TO_SOT_SMD:SOT-723" H 1650 1250 50  0001 C CNN
 F 3 "~" H 1450 1150 50  0001 C CNN
+F 4 "C415718" H 1450 1150 50  0001 C CNN "LCSC"
 	1    1450 1150
 	0    -1   -1   0
@@
 F 2 "Capacitor_SMD:C_0402_1005Metric" H 6900 1200 50  0001 C CNN
 F 3 "~" H 6900 1200 50  0001 C CNN
+F 4 "C15195" H 6900 1200 50  0001 C CNN "LCSC"
 	1    6900 1200
 	-1   0    0    1
@@
 P 6150 1200
 F 0 "C19" H 6242 1246 50  0000 L CNN
-F 1 "TBD" H 6242 1155 50  0000 L CNN
+F 1 "22uF" H 6242 1155 50  0000 L CNN
 F 2 "Capacitor_SMD:C_0603_1608Metric" H 6150 1200 50  0001 C CNN
 F 3 "~" H 6150 1200 50  0001 C CNN
+F 4 "C59461" H 6150 1200 50  0001 C CNN "LCSC"
 	1    6150 1200
 	1    0    0    -1
@@
 F 0 "FB1" V 5163 1050 50  0000 C CNN
 F 1 "100 @ 100MHz" V 5254 1050 50  0000 C CNN
-F 2 "Inductor_SMD:L_0402_1005Metric" V 5330 1050 50  0001 C CNN
+F 2 "Inductor_SMD:L_0805_2012Metric" V 5330 1050 50  0001 C CNN
 F 3 "~" H 5400 1050 50  0001 C CNN
+F 4 "C1017" H 5400 1050 50  0001 C CNN "LCSC"
 	1    5400 1050
 	0    1    1    0

Commit message: Minor changes
Parts:
- removed Q1, Q2: NTK3139P, Package_TO_SOT_SMD:SOT-723, symbol Device:Q_PMOS_GSD
- added Q1, Q2, Q3: AO3401A, Package_TO_SOT_SMD:SOT-23, symbol Transistor_FET:AO3401A
- added R11: 1M, Resistor_SMD:R_0402_1005Metric, symbol Device:R_Small
- added R12: 680, Resistor_SMD:R_0402_1005Metric, symbol Device:R_Small
- C12, C14: value 22pF -> 10pF; LCSC (none) -> C32949
- FB1: value 100 @ 100MHz -> 100Ohm@100MHz; LCSC C1017 -> C1015
- J2: footprint Connector_Coaxial:SMA_Samtec_SMA-J-P-H-ST-EM1_EdgeMount -> ak:SMA_Samtec_SMA-J-P-H-ST-EM1_EdgeMount
- R5: value TBD -> 1k; LCSC (none) -> C11702
- R8, R9: value TBD -> 680; LCSC (none) -> C25130
- U1: value Si7021-A20 -> SHT21; LCSC C132603 -> C84828
Connections:
- net BAT_LEVEL: now also U2.7 (PA1), R12.1; no longer U2.3 (PC15)
- net GND: now also Q2.1 (G), R12.2
- net LED_STATUS: now also U2.3 (PC15); no longer U2.7 (PA1)
- net NRF_PWR: now also Q1.1 (G)
- net VCC: now also Q1.2 (S), Q2.2 (S), Q3.2 (S), R11.1; no longer R8.1
- net at BT1.1 (+): now also Q2.3 (D)
- net at FB1.2: now also Q1.3 (D)
- net BAT_CHECK: now reaches U2.23 (PA15)
- net BAT_CHECK: now also Q3.1 (G), R11.2
- new net: Q3.3 (D), R8.1
- no-connect marks 11 -> 10
Other:
- note added: "Si7021 appears to be pin-compatible with SHT21"
- moved on the sheet: C19, FB1, R4, R5

Commit message: Minor changes
Parts:
- added C20: 100uF, Capacitor_Tantalum_SMD:CP_EIA-3528-15_AVX-H, symbol Device:CP_Small
- U1: value SHT21 -> SI7021; LCSC C84828 -> C132603
Connections:
- net +VSW: now also C20.1
- net GND: now also C20.2
Other:
- note removed: "Si7021 appears to be pin-compatible with SHT21"
- moved on the sheet: FB1, Q1, R4, R5
Changed lines of the file:
@@
 L Device:R_Small R5
 U 1 1 5F6EDFC5
-P 5500 1050
-F 0 "R5" V 5450 1200 50  0000 C CNN
-F 1 "1k" V 5450 900 50  0000 C CNN
-F 2 "Resistor_SMD:R_0402_1005Metric" H 5500 1050 50  0001 C CNN
-F 3 "~" H 5500 1050 50  0001 C CNN
-F 4 "C11702" H 5500 1050 50  0001 C CNN "LCSC"
-	1    5500 1050
+P 5350 1050
+F 0 "R5" V 5300 1200 50  0000 C CNN
+F 1 "1k" V 5300 900 50  0000 C CNN
+F 2 "Resistor_SMD:R_0402_1005Metric" H 5350 1050 50  0001 C CNN
+F 3 "~" H 5350 1050 50  0001 C CNN
+F 4 "C11702" H 5350 1050 50  0001 C CNN "LCSC"
+	1    5350 1050
 	0    1    1    0
 $EndComp
 Wire Wire Line
-	4650 1050 4900 1050
+	4500 1050 4750 1050
 Wire Wire Line
 	8150 1050 8250 1050
@@
 L Device:R_Small R4
 U 1 1 5F6FC380
-P 4050 1250
-F 0 "R4" H 4109 1296 50  0000 L CNN
-F 1 "1M" H 4109 1205 50  0000 L CNN
-F 2 "Resistor_SMD:R_0402_1005Metric" H 4050 1250 50  0001 C CNN
-F 3 "~" H 4050 1250 50  0001 C CNN
-F 4 "C26083" H 4050 1250 50  0001 C CNN "LCSC"
-	1    4050 1250
-	1    0    0    -1
-$EndComp
-Wire Wire Line
-	4050 1150 4050 1050
-Wire Wire Line
-	4050 1050 4250 1050
-Wire Wire Line
-	4050 1350 4050 1450
-Wire Wire Line
-	4450 1450 4450 1350
+P 3900 1250
+F 0 "R4" H 3959 1296 50  0000 L CNN
+F 1 "1M" H 3959 1205 50  0000 L CNN
+F 2 "Resistor_SMD:R_0402_1005Metric" H 3900 1250 50  0001 C CNN
+F 3 "~" H 3900 1250 50  0001 C CNN
+F 4 "C26083" H 3900 1250 50  0001 C CNN "LCSC"
+	1    3900 1250
+	1    0    0    -1
+$EndComp
+Wire Wire Line
+	3900 1150 3900 1050
+Wire Wire Line
+	3900 1050 4100 1050
+Wire Wire Line
+	3900 1350 3900 1450
+Wire Wire Line
+	4300 1450 4300 1350
 Wire Wire Line
 	5000 4550 5100 4550
@@
 	5000 4550 5000 4600
 Wire Wire Line
-	4050 1450 4450 1450
+	3900 1450 4300 1450
 Wire Wire Line
 	1900 4800 2350 4800
@@
 P 2300 2850
 F 0 "U1" H 2450 3100 50  0000 L CNN
-F 1 "SHT21" H 2450 2600 50  0000 L CNN
+F 1 "SI7021" H 2450 2600 50  0000 L CNN
 F 2 "Package_DFN_QFN:DFN-6-1EP_3x3mm_P1mm_EP1.5x2.4mm" H 2300 2450 50  0001 C CNN
 F 3 "https://www.silabs.com/documents/public/data-sheets/Si7021-A20.pdf" H 2100 3150 50  0001 C CNN
-F 4 "C84828" H 2300 2850 50  0001 C CNN "LCSC"
+F 4 "C132603" H 2300 2850 50  0001 C CNN "LCSC"
 	1    2300 2850
 	1    0    0    -1
@@
 	1350 5750 1400 5750
 Wire Wire Line
-	4050 950  4050 1050
-Connection ~ 4050 1050
+	3900 950  3900 1050
+Connection ~ 3900 1050
 Connection ~ 6450 1050
 Wire Wire Line
@@
 	6450 1050 6450 1100
 Wire Wire Line
-	5600 1050 6100 1050
+	5450 1050 5700 1050
 $Comp
 L Device:C_Small C8
@@
 $EndComp
 Wire Wire Line
-	4050 1450 3600 1450
-Connection ~ 4050 1450
+	3900 1450 3450 1450
+Connection ~ 3900 1450
 Connection ~ 2900 2400
 Wire Wire Line
@@
 Wire Wire Line
 	7800 5800 7800 5850
-Text Label 3600 1450 0    50   ~ 0
+Text Label 3450 1450 0    50   ~ 0
 NRF_PWR
 Wire Wire Line
@@
 L power:VCC #PWR016
 U 1 1 5F79FBFF
-P 4050 950
-F 0 "#PWR016" H 4050 800 50  0001 C CNN
-F 1 "VCC" H 4065 1123 50  0000 C CNN
-F 2 "" H 4050 950 50  0001 C CNN
-F 3 "" H 4050 950 50  0001 C CNN
-	1    4050 950
+P 3900 950
+F 0 "#PWR016" H 3900 800 50  0001 C CNN
+F 1 "VCC" H 3915 1123 50  0000 C CNN
+F 2 "" H 3900 950 50  0001 C CNN
+F 3 "" H 3900 950 50  0001 C CNN
+	1    3900 950
 	1    0    0    -1
 $EndComp
@@
 L Device:Ferrite_Bead_Small FB1
 U 1 1 5F7E119C
-P 5000 1050
-F 0 "FB1" V 4750 1050 50  0000 C CNN
-F 1 "100Ohm@100MHz" V 4854 1050 50  0000 C CNN
-F 2 "Inductor_SMD:L_0805_2012Metric" V 4930 1050 50  0001 C CNN
-F 3 "~" H 5000 1050 50  0001 C CNN
-F 4 "C1015" H 5000 1050 50  0001 C CNN "LCSC"
-	1    5000 1050
+P 4850 1050
+F 0 "FB1" V 4600 1050 50  0000 C CNN
+F 1 "100Ohm@100MHz" V 4704 1050 50  0000 C CNN
+F 2 "Inductor_SMD:L_0805_2012Metric" V 4780 1050 50  0001 C CNN
+F 3 "~" H 4850 1050 50  0001 C CNN
+F 4 "C1015" H 4850 1050 50  0001 C CNN "LCSC"
+	1    4850 1050
 	0    1    1    0
 $EndComp
 Wire Wire Line
-	5100 1050 5400 1050
+	4950 1050 5250 1050
 $Comp
 L power:PWR_FLAG #FLG0103
@@
 L Transistor_FET:AO3401A Q1
 U 1 1 5F790A3D
-P 4450 1150
-F 0 "Q1" V 4792 1150 50  0000 C CNN
-F 1 "AO3401A" V 4701 1150 50  0000 C CNN
-F 2 "Package_TO_SOT_SMD:SOT-23" H 4650 1075 50  0001 L CIN
-F 3 "http://www.aosmd.com/pdfs/datasheet/AO3401A.pdf" H 4450 1150 50  0001 L CNN
-F 4 "C15127" V 4450 1150 50  0001 C CNN "LCSC"
-	1    4450 1150
+P 4300 1150
+F 0 "Q1" V 4642 1150 50  0000 C CNN
+F 1 "AO3401A" V 4551 1150 50  0000 C CNN
+F 2 "Package_TO_SOT_SMD:SOT-23" H 4500 1075 50  0001 L CIN
+F 3 "http://www.aosmd.com/pdfs/datasheet/AO3401A.pdf" H 4300 1150 50  0001 L CNN
+F 4 "C15127" V 4300 1150 50  0001 C CNN "LCSC"
+	1    4300 1150
 	0    1    -1   0
 $EndComp
@@
 Wire Wire Line
 	8950 6100 8800 6100
-Text Notes 1400 3450 0    50   ~ 0
-Si7021 appears to be pin-compatible with SHT21
+$Comp
+L Device:CP_Small C20
+U 1 1 5F834F56
+P 5700 1200
+F 0 "C20" H 5788 1246 50  0000 L CNN
+F 1 "100uF" H 5788 1155 50  0000 L CNN
+F 2 "Capacitor_Tantalum_SMD:CP_EIA-3528-15_AVX-H" H 5700 1200 50  0001 C CNN
+F 3 "~" H 5700 1200 50  0001 C CNN
+F 4 "C16133" H 5700 1200 50  0001 C CNN "LCSC"
+	1    5700 1200
+	1    0    0    -1
+$EndComp
+Wire Wire Line
+	5700 1100 5700 1050
+Connection ~ 5700 1050
+Wire Wire Line
+	5700 1050 6100 1050
+$Comp
+L power:GND #PWR031
+U 1 1 5F843526
+P 5700 1300
+F 0 "#PWR031" H 5700 1050 50  0001 C CNN
+F 1 "GND" H 5705 1127 50  0001 C CNN
+F 2 "" H 5700 1300 50  0001 C CNN
+F 3 "" H 5700 1300 50  0001 C CNN
+	1    5700 1300
+	1    0    0    -1
+$EndComp
 $EndSCHEMATC
